File: pcb/Scanopcb.sch (EAGLE design)
At the start: 0 parts

Commit message: Added microcontroller
Parts:
- added IC1: MEGA8-P, atmel:MEGA8-P
- added R1: (no value), rcl:R-EU_0207/10
Changed lines of the file:
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@@
 <parts>
 <part name="FRAME1" library="frames" deviceset="A4L-LOC" device=""/>
+<part name="IC1" library="atmel" deviceset="MEGA8-P" device=""/>
+<part name="R1" library="rcl" deviceset="R-EU_" device="0207/10"/>
 </parts>
 <sheets>
@@
 <attribute name="SHEET" x="42.545" y="-2.54" size="2.54" layer="94"/>
 </instance>
+<instance part="IC1" gate="G$1" x="-129.54" y="119.38"/>
+<instance part="R1" gate="G$1" x="-162.56" y="147.32"/>
 </instances>
 <busses>

Commit message: WILLLIMS HEAD IS BIG
Parts:
- added R2, R3, R4: (no value), rcl:R-EU_0207/10
Changed lines of the file:
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@@
 <part name="IC1" library="atmel" deviceset="MEGA8-P" device=""/>
 <part name="R1" library="rcl" deviceset="R-EU_" device="0207/10"/>
+<part name="R2" library="rcl" deviceset="R-EU_" device="0207/10"/>
+<part name="R3" library="rcl" deviceset="R-EU_" device="0207/10"/>
+<part name="R4" library="rcl" deviceset="R-EU_" device="0207/10"/>
 </parts>
 <sheets>
@@
 <instance part="IC1" gate="G$1" x="-129.54" y="119.38"/>
 <instance part="R1" gate="G$1" x="-162.56" y="147.32"/>
+<instance part="R2" gate="G$1" x="-71.12" y="147.32"/>
+<instance part="R3" gate="G$1" x="-73.66" y="134.62"/>
+<instance part="R4" gate="G$1" x="-68.58" y="119.38"/>
 </instances>
 <busses>
